File: Schematics/Sr Design/Pan_and_Tilt.kicad_sch (KiCad schematic)
At the start: 3 parts, among them J2 Raspberry_Pi_4, M1 Motor_Servo, M2 Motor_Servo

Commit message: schematics updated
Changed lines of the file:
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@@
-	)
-	(symbol
-		(lib_id "power:+12V")
-		(at 193.04 66.04 0)
-		(unit 1)
-		(exclude_from_sim no)
-		(in_bom yes)
-		(on_board yes)
-		(dnp no)
-		(fields_autoplaced yes)
-		(property "Reference" "#PWR09"
-			(at 193.04 69.85 0)
-			(effects
-				(font
-					(size 1.27 1.27)
-				)
-				(hide yes)
-			)
-		)
-		(property "Value" "+12V"
-			(at 193.04 60.96 0)
-			(effects
-				(font
-					(size 1.27 1.27)
-				)
-			)
-		)
-		(property "Footprint" ""
-			(at 193.04 66.04 0)
-			(effects
-				(font
-					(size 1.27 1.27)
-				)
-				(hide yes)
-			)
-		)
-		(property "Datasheet" ""
-			(at 193.04 66.04 0)
-			(effects
-				(font
-					(size 1.27 1.27)
-				)
-				(hide yes)
-			)
-		)
-		(property "Description" "Power symbol creates a global label with name \"+12V\""
-			(at 193.04 66.04 0)
-			(effects
-				(font
-					(size 1.27 1.27)
-				)
-				(hide yes)
-			)
-		)
-		(pin "1"
-		)
-		(instances
-			(project ""
-				(path "/a9415093-c716-43d5-965a-b0cfe44093a0/2cead76a-a95c-4d3f-870e-84fb66109598"
-					(reference "#PWR09")
-					(unit 1)
-				)
-			)
-		)
 	)
 	(symbol

Commit message: scematics update
Parts:
- removed J2: Raspberry_Pi_4, symbol Connector:Raspberry_Pi_4
- removed M1, M2: Motor_Servo, symbol Motor:Motor_Servo
- added J1: GPIO 21, Connector_PinHeader_1.00mm:PinHeader_1x01_P1.00mm_Vertical, symbol Connector:Conn_01x01_Socket
- added J10: GPIO 20, Connector_PinHeader_1.00mm:PinHeader_1x01_P1.00mm_Vertical, symbol Connector:Conn_01x01_Socket
- added J11: Pan GPIO, Connector_PinHeader_1.00mm:PinHeader_1x01_P1.00mm_Vertical, symbol Connector:Conn_01x01_Socket
- added J12: Pan GND, Connector_PinHeader_1.00mm:PinHeader_1x01_P1.00mm_Vertical, symbol Connector:Conn_01x01_Socket
- added J13: Tilt 5V, Connector_PinHeader_1.00mm:PinHeader_1x01_P1.00mm_Vertical, symbol Connector:Conn_01x01_Socket
- added J14: Tilt GPIO, Connector_PinHeader_1.00mm:PinHeader_1x01_P1.00mm_Vertical, symbol Connector:Conn_01x01_Socket
- added J15: Tilt GND, Connector_PinHeader_1.00mm:PinHeader_1x01_P1.00mm_Vertical, symbol Connector:Conn_01x01_Socket
- added J2: Pan 5V, Connector_PinHeader_1.00mm:PinHeader_1x01_P1.00mm_Vertical, symbol Connector:Conn_01x01_Socket
Connections:
- net GND: now also J12.1 (Pin_1), J15.1 (Pin_1)
- new net: J10.1 (Pin_1), J11.1 (Pin_1)
- new net: J1.1 (Pin_1), J14.1 (Pin_1)
- new net +7V: J13.1 (Pin_1), J2.1 (Pin_1)
