File: Schematics/Sr Design/Water Gun.kicad_sch (KiCad schematic)
At the start: 8 parts, among them J1 Raspberry_Pi_4, Q1 C6144, Q2 C6144

Commit message: scematics update
Parts:
- removed J1: Raspberry_Pi_4, symbol Connector:Raspberry_Pi_4
- added J8: GPIO 23, Connector_PinHeader_1.00mm:PinHeader_1x01_P1.00mm_Vertical, symbol Connector:Conn_01x01_Socket
- added J9: GPIO 24, Connector_PinHeader_1.00mm:PinHeader_1x01_P1.00mm_Vertical, symbol Connector:Conn_01x01_Socket
- R1, R2: footprint (none) -> Resistor_SMD:R_0201_0603Metric
- U1, U2: footprint (none) -> Connector_PinHeader_1.00mm:PinHeader_1x02_P1.00mm_Vertical
Connections:
- net at R2.1: now also J9.1 (Pin_1)
- net at R1.1: now also J8.1 (Pin_1)
Changed lines of the file:
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@@
 	(wire
 		(pts
-			(xy 189.23 62.23) (xy 189.23 87.63)
+			(xy 189.23 62.23) (xy 189.23 91.44)
 		)
 		(stroke
@@
 	(wire
 		(pts
-			(xy 189.23 87.63) (xy 91.44 87.63)
+			(xy 189.23 91.44) (xy 91.44 91.44)
 		)
 		(stroke
@@
 			)
 		)
-		(property "Footprint" ""
+		(property "Footprint" "Resistor_SMD:R_0201_0603Metric"
 			(at 193.294 61.214 90)
 			(effects
@@
 	)
 	(symbol
+		(lib_id "Connector:Conn_01x01_Socket")
+		(at 86.36 91.44 180)
+		(unit 1)
+		(exclude_from_sim no)
+		(in_bom yes)
+		(on_board yes)
+		(dnp no)
+		(property "Reference" "J9"
+			(at 80.518 93.472 0)
+			(effects
+				(font
+					(size 1.27 1.27)
+				)
+			)
+		)
+		(property "Value" "GPIO 24"
+			(at 81.026 91.44 0)
+			(effects
+				(font
+					(size 1.27 1.27)
+				)
+			)
+		)
+		(property "Footprint" "Connector_PinHeader_1.00mm:PinHeader_1x01_P1.00mm_Vertical"
+			(at 86.36 91.44 0)
+			(effects
+				(font
+					(size 1.27 1.27)
+				)
+				(hide yes)
+			)
+		)
+		(property "Datasheet" "~"
+			(at 86.36 91.44 0)
+			(effects
+				(font
+					(size 1.27 1.27)
+				)
+				(hide yes)
+			)
+		)
+		(property "Description" "Generic connector, single row, 01x01, script generated"
+			(at 86.36 91.44 0)
+			(effects
+				(font
+					(size 1.27 1.27)
+				)
+				(hide yes)
+			)
+		)
+		(pin "1"
+		)
+		(instances
+			(project ""
+				(path "/a9415093-c716-43d5-965a-b0cfe44093a0/1c7459dd-cf78-4d64-bcbe-5c11431f21c6"
+					(reference "J9")
+					(unit 1)
+				)
+			)
+		)
+	)
+	(symbol
 		(lib_id "Water Gun:Pump")
 		(at 119.38 45.72 270)
@@
 			)
 		)
-		(property "Footprint" ""
+		(property "Footprint" "Connector_PinHeader_1.00mm:PinHeader_1x02_P1.00mm_Vertical"
 			(at 119.38 45.72 0)
 			(effects
@@
 			)
 		)
-		(property "Footprint" ""
+		(property "Footprint" "Connector_PinHeader_1.00mm:PinHeader_1x02_P1.00mm_Vertical"
 			(at 199.39 45.72 0)
 			(effects
@@
 	)
 	(symbol
+		(lib_id "Connector:Conn_01x01_Socket")
+		(at 86.36 85.09 180)
+		(unit 1)
+		(exclude_from_sim no)
+		(in_bom yes)
+		(on_board yes)
+		(dnp no)
+		(property "Reference" "J8"
+			(at 79.756 86.868 0)
+			(effects
+				(font
+					(size 1.27 1.27)
+				)
+			)
+		)
+		(property "Value" "GPIO 23"
+			(at 79.756 84.836 0)
+			(effects
+				(font
+					(size 1.27 1.27)
+				)
+			)
+		)
+		(property "Footprint" "Connector_PinHeader_1.00mm:PinHeader_1x01_P1.00mm_Vertical"
+			(at 86.36 85.09 0)
+			(effects
+				(font
+					(size 1.27 1.27)
+				)
+				(hide yes)
+			)
+		)
+		(property "Datasheet" "~"
+			(at 86.36 85.09 0)
+			(effects
+				(font
+					(size 1.27 1.27)
+				)
+				(hide yes)
+			)
+		)
+		(property "Description" "Generic connector, single row, 01x01, script generated"
+			(at 86.36 85.09 0)
+			(effects
+				(font
+					(size 1.27 1.27)
+				)
+				(hide yes)
+			)
+		)
+		(pin "1"
+		)
+		(instances
+			(project ""
+				(path "/a9415093-c716-43d5-965a-b0cfe44093a0/1c7459dd-cf78-4d64-bcbe-5c11431f21c6"
+					(reference "J8")
+					(unit 1)
+				)
+			)
+		)
+	)
+	(symbol
 		(lib_id "power:+12V")
 		(at 124.46 38.1 0)
@@
 	)
 	(symbol
-		(lib_id "Connector:Raspberry_Pi_4")
-		(at 58.42 72.39 0)
-		(mirror y)
-		(unit 1)
-		(exclude_from_sim no)
-		(in_bom yes)
-		(on_board yes)
-		(dnp no)
-		(property "Reference" "J1"
-			(at 58.42 41.91 0)
-			(effects
-				(font
-					(size 1.27 1.27)
-				)
-			)
-		)
-		(property "Value" "Raspberry_Pi_4"
-			(at 58.42 44.45 0)
-			(effects
-				(font
-					(size 1.27 1.27)
-				)
-			)
-		)
-		(property "Footprint" ""
-			(at -11.684 119.888 0)
-			(effects
-				(font
-					(size 1.27 1.27)
-				)
-				(justify left)
-				(hide yes)
-			)
-		)
-		(property "Datasheet" "https://datasheets.raspberrypi.com/rpi4/raspberry-pi-4-datasheet.pdf"
-			(at 42.672 104.648 0)
-			(effects
-				(font
-					(size 1.27 1.27)
-				)
-				(justify left)
-				(hide yes)
-			)
-		)
-		(property "Description" "Raspberry Pi 4 Model B"
-			(at 42.672 102.108 0)
-			(effects
-				(font
-					(size 1.27 1.27)
-				)
-				(justify left)
-				(hide yes)
-			)
-		)
-		(pin "32"
-		)
-		(pin "8"
-		)
-		(pin "10"
-		)
-		(pin "12"
-		)
-		(pin "38"
-		)
-		(pin "40"
-		)
-		(pin "33"
-		)
-		(pin "36"
-		)
-		(pin "11"
-		)
-		(pin "35"
-		)
-		(pin "28"
-		)
-		(pin "6"
-		)
-		(pin "13"
-		)
-		(pin "31"
-		)
-		(pin "24"
-		)
-		(pin "18"
-		)
-		(pin "20"
-		)
-		(pin "25"
-		)
-		(pin "22"
-		)
-		(pin "2"
-		)
-		(pin "16"
-		)
-		(pin "37"
-		)
-		(pin "14"
-		)
-		(pin "34"
-		)
-		(pin "39"
-		)
-		(pin "15"
-		)
-		(pin "9"
-		)
-		(pin "30"
-		)
-		(pin "4"
-		)
-		(pin "1"
-		)
-		(pin "17"
-		)
-		(pin "27"
-		)
-		(pin "3"
-		)
-		(pin "5"
-		)
-		(pin "7"
-		)
-		(pin "29"
-		)
-		(pin "26"
-		)
-		(pin "19"
-		)
-		(pin "21"
-		)
-		(pin "23"
-		)
-		(instances
-			(project ""
-				(path "/a9415093-c716-43d5-965a-b0cfe44093a0/1c7459dd-cf78-4d64-bcbe-5c11431f21c6"
-					(reference "J1")
-					(unit 1)
-				)
-			)
-		)
-	)
-	(symbol
 		(lib_id "power:GND")
 		(at 204.47 72.39 0)
@@
 			)
 		)
-		(property "Footprint" ""
+		(property "Footprint" "Resistor_SMD:R_0201_0603Metric"
 			(at 108.204 61.214 90)
 			(effects
