File: Schematics/Sr Design/Water Sensor_sch.kicad_sch (KiCad schematic)
At the start: 5 parts, among them J5 Tanner's Capacitor, U5 LM555CN

Commit message: scematics update
Parts:
- removed U5: LM555CN, LM555CN:DIP254P762X533-8, symbol LM555CN:LM555CN
- added C1: 1u F, Capacitor_SMD:C_0201_0603Metric, symbol Device:C
- added D2: LED, LED_SMD:LED_0201_0603Metric, symbol Device:LED
- added J16: GPIO 20, Connector_PinHeader_1.00mm:PinHeader_1x01_P1.00mm_Vertical, symbol Connector:Conn_01x01_Socket
- added J6: Water Float Switch, Connector_PinHeader_1.00mm:PinHeader_1x02_P1.00mm_Vertical, symbol Connector:Conn_01x02_Socket
- added J7: GPIO 22, Connector_PinHeader_1.00mm:PinHeader_1x01_P1.00mm_Vertical, symbol Connector:Conn_01x01_Socket
- added R6: 330, Resistor_SMD:R_0201_0603Metric, symbol Device:R_US
- added U6: LM555CN, LM555CN:DIP762W46P254L960H508Q8, symbol LM555CN:LM555CN
- J5: footprint (none) -> Connector_PinHeader_1.00mm:PinHeader_1x02_P1.00mm_Vertical
- R3, R4, R5: footprint (none) -> Resistor_SMD:R_0201_0603Metric
Connections:
- net +12V: now also U6.8 (VCC)
- net GND: now also C1.2, D2.1 (K), U6.1 (GND)
- net at R3.2, R4.1: now also U6.4 (RESET), U6.7 (DISCH)
- net at R5.1: now also J16.1 (Pin_1), U6.3 (OUT)
- net at J5.1 (Pin_1), R4.2: now also J6.2 (Pin_2), U6.2 (TRIGGER), U6.6 (THR)
- new net: J7.1 (Pin_1), R6.1
- new net: D2.2 (A), R6.2
- new net: C1.1, J6.1 (Pin_1)
Other:
- moved on the sheet: J5, R3, R4, R5
